File: beta/hardware/lr8i2c/LONG_8_REL_I2C_beta1/8_relays_i2c.sch (KiCad schematic (older format))
At the start: 91 parts, among them K1 CONN_3, K10 G5LA-1-12VDC, K11 CONN_3, K12 CONN_3, K13 CONN_3, K14 CONN_3, K15 CONN_3, K16 CONN_3, K17 CONN_3, K18 CONN_3, K2 CONN_3, K3 G5LA-1-12VDC, K4 G5LA-1-12VDC, K5 G5LA-1-12VDC, K6 G5LA-1-12VDC, K7 G5LA-1-12VDC, K8 G5LA-1-12VDC, K9 G5LA-1-12VDC, P1 CONN_10, P2 CONN_6, Q1 PNP, Q10 DSS20201L NPN, Q11 DSS20201L NPN, Q12 DSS20201L NPN, Q13 DSS20201L NPN, Q14 DSS20201L NPN, Q15 DSS20201L NPN, Q16 DSS20201L NPN, Q2 PNP, Q3 PNP, Q4 PNP, Q5 PNP, Q6 PNP, Q7 PNP, Q8 PNP, Q9 DSS20201L NPN, U1 PCF8574

Commit message: routage en cours
Parts:
- added P112: CONN_6, symbol CONN_6
- renumbered D1 to D101, D2 to D102, D3 to D103, D4 to D104, D5 to D105, D6 to D106, D7 to D107, D8 to D108, D9 to D109, D10 to D110, D11 to D111, D12 to D112, D13 to D113, D14 to D114, D15 to D115, D16 to D116, K3 to K101, K4 to K102, K5 to K103, K6 to K104, K7 to K105, K8 to K106, K9 to K107, K10 to K108, K11 to P101, K12 to P102, K13 to P103, K14 to P104, K15 to P105, K16 to P106, K17 to P107, K18 to P108, K1 to P109, P2 to P110, K2 to P111, P1 to P113, Q1 to Q101, Q2 to Q102, Q3 to Q103, Q4 to Q104, Q5 to Q105, Q6 to Q106, Q7 to Q107, Q8 to Q108, Q9 to Q109, Q10 to Q110, Q11 to Q111, Q12 to Q112, Q13 to Q113, Q14 to Q114, Q15 to Q115, Q16 to Q116, R1 to R101, R2 to R102, R3 to R103, R4 to R104, R5 to R105, R6 to R106, R7 to R107, R8 to R108, R9 to R109, R10 to R110, R11 to R111, R12 to R112, R13 to R113, R14 to R114, R15 to R115, R16 to R116, R17 to R117, R18 to R118, R19 to R119, R20 to R120, R21 to R121, R22 to R122, R23 to R123, R24 to R124, R25 to R125, R26 to R126, R27 to R127, R28 to R128, R29 to R129, R30 to R130, R31 to R131, R32 to R132, R33 to R133, R34 to R134, R35 to R135, U1 to U101
Connections:
- net +5V: now also P112.1
- net /INT: now also P112.5
- net GND: now also P112.2
- net SCL: now also P112.3
- net SDA: now also P112.4
- net spare: now also P112.6
- net CMD0: now reaches R104.1, U101.4 (P0)
- net CMD5: now reaches R109.1, U101.10 (P5)
- net CMD6: now reaches R110.1, U101.11 (P6)
- net CMD7: now reaches R111.1, U101.12 (P7)
- net CMD1: now reaches R105.1, U101.5 (P1)
- net CMD2: now reaches R106.1, U101.6 (P2)
- net CMD3: now reaches R107.1, U101.7 (P3)
- net CMD4: now reaches R108.1, U101.9 (P4)
Other:
- moved on the sheet: P109, P110, P111, P113

Commit message: routage suite
Parts:
- removed P113: CONN_10, symbol CONN_10
Changed lines of the file:
@@
-EESchema Schematic File Version 2  date mer. 18 avril 2012 13:06:07 CEST
+EESchema Schematic File Version 2  date mer. 18 avril 2012 20:39:17 CEST
 LIBS:power
 LIBS:device
@@
 Text Label 13250 3450 2    60   ~ 0
 spare
-Text Label 15350 4150 0    60   ~ 0
-OUT0
-Text Label 15350 3450 0    60   ~ 0
-OUT7
-Text Label 15350 3550 0    60   ~ 0
-OUT6
-Text Label 15350 3650 0    60   ~ 0
-OUT5
-Text Label 15350 3750 0    60   ~ 0
-OUT4
-Text Label 15350 3850 0    60   ~ 0
-OUT3
-Text Label 15350 3950 0    60   ~ 0
-OUT2
-Text Label 15350 4050 0    60   ~ 0
-OUT1
-$Comp
-L CONN_10 P113
-U 1 1 4F8DBB08
-P 15000 3700
-F 0 "P113" V 14950 3700 60  0000 C CNN
-F 1 "CONN_10" V 15050 3700 60  0000 C CNN
-	1    15000 3700
-	-1   0    0    1
-$EndComp
 Text Label 8200 10350 2    60   ~ 0
 OUT7
