File: beta/hardware/smb/v0.0/uSD_card.sch (KiCad schematic (older format))
At the start: 6 parts

Commit message: few modifications
Parts:
- gave numbers to parts that had none: 6
Changed lines of the file:
@@
-EESchema Schematic File Version 2  date 01/07/2012 20:02:11
+EESchema Schematic File Version 2  date 01/07/2012 23:30:37
 LIBS:power
 LIBS:device
@@
 	2675 3800 2675 800
 Wire Notes Line
-	1150 3800 2675 3800
+	2675 3800 1150 3800
 Wire Notes Line
 	1150 3800 1150 800
@@
 SPI_MISO
 $Comp
-L GND #PWR?
+L GND #PWR208
 U 1 1 4FF08F4C
 P 2100 3675
-F 0 "#PWR?" H 2100 3675 30  0001 C CNN
+F 0 "#PWR208" H 2100 3675 30  0001 C CNN
 F 1 "GND" H 2100 3605 30  0001 C CNN
 	1    2100 3675
@@
 $EndComp
 $Comp
-L +5V #PWR?
+L +5V #PWR207
 U 1 1 4FF08F3A
 P 2100 3275
-F 0 "#PWR?" H 2100 3365 20  0001 C CNN
+F 0 "#PWR207" H 2100 3365 20  0001 C CNN
 F 1 "+5V" H 2100 3365 30  0000 C CNN
 	1    2100 3275
@@
 $EndComp
 $Comp
-L 74LVC1G126GW U?
+L 74LVC1G126GW U206
 U 1 1 4FF08F14
 P 2000 3525
-F 0 "U?" H 2275 3400 60  0000 C CNN
+F 0 "U206" H 2275 3400 60  0000 C CNN
 F 1 "74LVC1G126GW" H 1600 3575 60  0000 C CNN
 	1    2000 3525
@@
 SPI_CLK
 $Comp
-L GND #PWR?
+L GND #PWR206
 U 1 1 4FF08D9D
 P 2100 2750
-F 0 "#PWR?" H 2100 2750 30  0001 C CNN
+F 0 "#PWR206" H 2100 2750 30  0001 C CNN
 F 1 "GND" H 2100 2680 30  0001 C CNN
 	1    2100 2750
@@
 $EndComp
 $Comp
-L +3.3V #PWR?
+L +3.3V #PWR205
 U 1 1 4FF08D91
 P 2100 2350
-F 0 "#PWR?" H 2100 2310 30  0001 C CNN
+F 0 "#PWR205" H 2100 2310 30  0001 C CNN
 F 1 "+3.3V" H 2100 2460 30  0000 C CNN
 	1    2100 2350
@@
 $EndComp
 $Comp
-L 74LVC1G126GW U?
+L 74LVC1G126GW U205
 U 1 1 4FF08D87
 P 2000 2600
-F 0 "U?" H 2275 2475 60  0000 C CNN
+F 0 "U205" H 2275 2475 60  0000 C CNN
 F 1 "74LVC1G126GW" H 1600 2650 60  0000 C CNN
 	1    2000 2600
@@
 CLK_33
 $Comp
-L +3.3V #PWR?
+L +3.3V #PWR203
 U 1 1 4FF07933
 P 2100 1725
-F 0 "#PWR?" H 2100 1685 30  0001 C CNN
+F 0 "#PWR203" H 2100 1685 30  0001 C CNN
 F 1 "+3.3V" H 2100 1835 30  0000 C CNN
 	1    2100 1725
@@
 $EndComp
 $Comp
-L GND #PWR?
+L GND #PWR204
 U 1 1 4FF0791F
 P 2100 2125
-F 0 "#PWR?" H 2100 2125 30  0001 C CNN
+F 0 "#PWR204" H 2100 2125 30  0001 C CNN
 F 1 "GND" H 2100 2055 30  0001 C CNN
 	1    2100 2125
@@
 MOSI_33
 $Comp
-L GND #PWR?
+L GND #PWR202
 U 1 1 4FF077F6
 P 2100 1525
-F 0 "#PWR?" H 2100 1525 30  0001 C CNN
+F 0 "#PWR202" H 2100 1525 30  0001 C CNN
 F 1 "GND" H 2100 1455 30  0001 C CNN
 	1    2100 1525
@@
 CS_33
 $Comp
-L 74LVC1G126GW U?
+L 74LVC1G126GW U204
 U 1 1 4FF07749
 P 2000 1975
-F 0 "U?" H 2275 1850 60  0000 C CNN
+F 0 "U204" H 2275 1850 60  0000 C CNN
 F 1 "74LVC1G126GW" H 1600 2025 60  0000 C CNN
 	1    2000 1975
@@
 uSD_CS
 $Comp
-L +3.3V #PWR?
+L +3.3V #PWR201
 U 1 1 4FF0764D
 P 2100 1125
-F 0 "#PWR?" H 2100 1085 30  0001 C CNN
+F 0 "#PWR201" H 2100 1085 30  0001 C CNN
 F 1 "+3.3V" H 2100 1235 30  0000 C CNN
 	1    2100 1125
@@
 $EndComp
 $Comp
-L 74LVC1G126GW U?
+L 74LVC1G126GW U203
 U 1 1 4FF07632
 P 2000 1375
-F 0 "U?" H 2275 1250 60  0000 C CNN
+F 0 "U203" H 2275 1250 60  0000 C CNN
 F 1 "74LVC1G126GW" H 1600 1425 60  0000 C CNN
 	1    2000 1375
@@
 $EndComp
 $Comp
-L +3.3V #PWR?
+L +3.3V #PWR209
 U 1 1 4FF06B96
 P 3575 2075
-F 0 "#PWR?" H 3575 2035 30  0001 C CNN
+F 0 "#PWR209" H 3575 2035 30  0001 C CNN
 F 1 "+3.3V" H 3575 2185 30  0000 C CNN
 	1    3575 2075
@@
 $EndComp
 $Comp
-L CSMALL C?
+L CSMALL C215
 U 1 1 4FF06B5D
 P 3575 2650
-F 0 "C?" H 3600 2700 30  0000 L CNN
+F 0 "C215" H 3600 2700 30  0000 L CNN
 F 1 "0.1uF" V 3500 2600 30  0000 L CNN
 	1    3575 2650
@@
 $EndComp
 $Comp
-L GND #PWR?
+L GND #PWR210
 U 1 1 4FF06B3E
 P 3575 2800
-F 0 "#PWR?" H 3575 2800 30  0001 C CNN
+F 0 "#PWR210" H 3575 2800 30  0001 C CNN
 F 1 "GND" H 3575 2730 30  0001 C CNN
 	1    3575 2800
@@
 $EndComp
 $Comp
-L USD_CONN J?
+L USD_CONN J202
 U 1 1 4FF052FB
 P 3900 2300
-F 0 "J?" H 4100 2125 60  0000 C CNN
+F 0 "J202" H 4100 2125 60  0000 C CNN
 F 1 "USD_CONN" H 3950 2575 60  0000 C CNN
 	1    3900 2300

Commit message: New components and corrections
Parts:
- C215: footprint (none) -> SM0603
- J202: footprint (none) -> DM3CS-SF
- U203, U204, U205, U206: footprint (none) -> SOT353
Changed lines of the file:
@@
-EESchema Schematic File Version 2  date 01/07/2012 23:30:37
+EESchema Schematic File Version 2  date 14/07/2012 20:45:27
 LIBS:power
 LIBS:device
@@
 LIBS:usd_conn
 LIBS:74lvc1g126gw
+LIBS:dual_self
 LIBS:SMB-cache
 EELAYER 25  0
@@
 Sheet 2 4
 Title ""
-Date "1 jul 2012"
+Date "14 jul 2012"
 Rev ""
 Comp ""
@@
 SPI_MISO
 $Comp
-L GND #PWR208
+L GND #PWR023
 U 1 1 4FF08F4C
 P 2100 3675
-F 0 "#PWR208" H 2100 3675 30  0001 C CNN
+F 0 "#PWR023" H 2100 3675 30  0001 C CNN
 F 1 "GND" H 2100 3605 30  0001 C CNN
 	1    2100 3675
@@
 $EndComp
 $Comp
-L +5V #PWR207
+L +5V #PWR024
 U 1 1 4FF08F3A
 P 2100 3275
-F 0 "#PWR207" H 2100 3365 20  0001 C CNN
+F 0 "#PWR024" H 2100 3365 20  0001 C CNN
 F 1 "+5V" H 2100 3365 30  0000 C CNN
 	1    2100 3275
@@
 F 0 "U206" H 2275 3400 60  0000 C CNN
 F 1 "74LVC1G126GW" H 1600 3575 60  0000 C CNN
+F 2 "SOT353" H 1600 3675 60  0000 C CNN
 	1    2000 3525
 	1    0    0    -1
@@
 SPI_CLK
 $Comp
-L GND #PWR206
+L GND #PWR025
 U 1 1 4FF08D9D
 P 2100 2750
-F 0 "#PWR206" H 2100 2750 30  0001 C CNN
+F 0 "#PWR025" H 2100 2750 30  0001 C CNN
 F 1 "GND" H 2100 2680 30  0001 C CNN
 	1    2100 2750
@@
 $EndComp
 $Comp
-L +3.3V #PWR205
+L +3.3V #PWR026
 U 1 1 4FF08D91
 P 2100 2350
-F 0 "#PWR205" H 2100 2310 30  0001 C CNN
+F 0 "#PWR026" H 2100 2310 30  0001 C CNN
 F 1 "+3.3V" H 2100 2460 30  0000 C CNN
 	1    2100 2350
@@
 F 0 "U205" H 2275 2475 60  0000 C CNN
 F 1 "74LVC1G126GW" H 1600 2650 60  0000 C CNN
+F 2 "SOT353" H 1600 2750 60  0000 C CNN
 	1    2000 2600
 	1    0    0    -1
@@
 CLK_33
 $Comp
-L +3.3V #PWR203
+L +3.3V #PWR027
 U 1 1 4FF07933
 P 2100 1725
-F 0 "#PWR203" H 2100 1685 30  0001 C CNN
+F 0 "#PWR027" H 2100 1685 30  0001 C CNN
 F 1 "+3.3V" H 2100 1835 30  0000 C CNN
 	1    2100 1725
@@
 $EndComp
 $Comp
-L GND #PWR204
+L GND #PWR028
 U 1 1 4FF0791F
 P 2100 2125
-F 0 "#PWR204" H 2100 2125 30  0001 C CNN
+F 0 "#PWR028" H 2100 2125 30  0001 C CNN
 F 1 "GND" H 2100 2055 30  0001 C CNN
 	1    2100 2125
@@
 MOSI_33
 $Comp
-L GND #PWR202
+L GND #PWR029
 U 1 1 4FF077F6
 P 2100 1525
-F 0 "#PWR202" H 2100 1525 30  0001 C CNN
+F 0 "#PWR029" H 2100 1525 30  0001 C CNN
 F 1 "GND" H 2100 1455 30  0001 C CNN
 	1    2100 1525
@@
 F 0 "U204" H 2275 1850 60  0000 C CNN
 F 1 "74LVC1G126GW" H 1600 2025 60  0000 C CNN
+F 2 "SOT353" H 1600 2125 60  0000 C CNN
 	1    2000 1975
 	1    0    0    -1
@@
 uSD_CS
 $Comp
-L +3.3V #PWR201
+L +3.3V #PWR030
 U 1 1 4FF0764D
 P 2100 1125
-F 0 "#PWR201" H 2100 1085 30  0001 C CNN
+F 0 "#PWR030" H 2100 1085 30  0001 C CNN
 F 1 "+3.3V" H 2100 1235 30  0000 C CNN
 	1    2100 1125
@@
 F 0 "U203" H 2275 1250 60  0000 C CNN
 F 1 "74LVC1G126GW" H 1600 1425 60  0000 C CNN
+F 2 "SOT353" H 1600 1525 60  0000 C CNN
 	1    2000 1375
 	1    0    0    -1
 $EndComp
 $Comp
-L +3.3V #PWR209
+L +3.3V #PWR031
 U 1 1 4FF06B96
 P 3575 2075
-F 0 "#PWR209" H 3575 2035 30  0001 C CNN
+F 0 "#PWR031" H 3575 2035 30  0001 C CNN
 F 1 "+3.3V" H 3575 2185 30  0000 C CNN
 	1    3575 2075
@@
 F 0 "C215" H 3600 2700 30  0000 L CNN
 F 1 "0.1uF" V 3500 2600 30  0000 L CNN
+F 2 "SM0603" V 3600 2600 30  0000 C CNN
 	1    3575 2650
 	-1   0    0    1
 $EndComp
 $Comp
-L GND #PWR210
+L GND #PWR032
 U 1 1 4FF06B3E
 P 3575 2800
-F 0 "#PWR210" H 3575 2800 30  0001 C CNN
+F 0 "#PWR032" H 3575 2800 30  0001 C CNN
 F 1 "GND" H 3575 2730 30  0001 C CNN
 	1    3575 2800
@@
 F 0 "J202" H 4100 2125 60  0000 C CNN
 F 1 "USD_CONN" H 3950 2575 60  0000 C CNN
+F 2 "DM3CS-SF" H 3950 2675 60  0000 C CNN
 	1    3900 2300
 	1    0    0    -1
